File: hardware/纠编机/纠编机.kicad_sch (KiCad schematic)
At the start: 50 parts

Commit message: 完善原理图的绘制
Parts:
- added AE1: Antenna, symbol Device:Antenna
- added C13, C14, C15: 10uf/50v, symbol Device:C
- added C16: 1pf, symbol Device:C
- added C17: 0.5pf, symbol Device:C
- added C4: 22uf/50v, symbol Device:C
- added D10, D8, D9: 5819, symbol Device:D
- added D11, D13: R_LED, symbol Device:LED
- added D12: G_LED, symbol Device:LED
- added L2: 1NH, symbol Device:L
- added Q2, Q3, Q5, Q6, Q7, Q8: NMOS, symbol Simulation_SPICE:NMOS
- added R27, R37, R44: 1K, symbol Device:R
- added R28, R42: 5mR, symbol Device:R
- added R29, R32, R33, R34, R38, R39: 22R, symbol Device:R
- added R30, R31, R35, R36, R40, R41: 10K, symbol Device:R
- added R43: 0R, symbol Device:R
- added U4: TSSOP20, symbol Driver_Motor:FD6288_TSSOP20
- added U5: TSSOP20, symbol RF2G4_sym:DCT5805_TSSOP20
- added Y1: 24MHz 10ppm, symbol Device:Crystal
- U1: footprint (none) -> QFN32
- U2: value ~ -> 6209
- U3: value ~ -> ESOP8
Connections:
- net IR_U_N is gone; now on net -BATT: R2.1
- net IR_V_N is gone; now on net -BATT: R3.1
- net MCU_GND is gone; now on net -BATT: U1.5 (VSS)
- net +12V: now also C4.1, D10.2 (A), D8.2 (A), D9.2 (A), U4.7 (VCC)
- net +BATT: now also Q2.1 (D), Q5.1 (D), Q7.1 (D)
- net -BATT: now also C10.2, C11.2, C12.2, C6.2, C7.2, C8.2, C9.2, D6.2 (A), D7.2 (A), NTC1.2, NTC2.2, R13.2, R18.2, R19.2, R20.2, R24.1, R26.2, U2. (VOut), C16.1, C17.2, C4.2, Q6.3 (S), R28.1, R31.2, R35.2, R40.2, R42.1, R43.1, U4.8 (COM), U5.18 (VSS), Y1.2
- net Enable: now also U5.2 (PB4)
- net IR_U: now also Q3.3 (S), R28.2
- net IR_V: now also Q8.3 (S), R42.2
- net U_HIN: now also U4.1 (HIN1)
- net U_LIN: now also U4.4 (LIN1)
- net U_Out: now also C13.2, Q2.3 (S), Q3.1 (D), R30.2, U4.18 (VS1)
- net UartRX: now also D12.1 (K), U5.9 (PA3)
- net UartTX: now also D11.1 (K), U5.10 (PA4)
- net VDD_3.3v: now also R27.2, R37.2, R44.1, U5.17 (VDD)
- net V_HIN: now also U4.2 (HIN2)
- net V_LIN: now also U4.5 (LIN2)
- net V_Out: now also C14.2, Q7.3 (S), Q8.1 (D), R41.2, U4.15 (VS2)
- net W_HIN: now also U4.3 (HIN3)
- net W_LIN: now also U4.6 (LIN3)
- net W_Out: now also C15.2, Q5.3 (S), Q6.1 (D), R36.2, U4.12 (VS3)
- net direct: now also U5.4 (PB2)
- net speed_IN: now also U5.3 (PB3)
- removed net GNDREF: C10.2, C11.2, C12.2, C6.2, C7.2, C8.2, C9.2, D6.2 (A), D7.2 (A), NTC1.2, NTC2.2, R13.2, R18.2, R19.2, R20.2, R24.1, R26.2, U2. (VOut)
- new net: C16.2, L2.1, U5.20 (ANT)
- new net: AE1.1 (A), C17.1, L2.2
- new net: D13.1 (K), U5.11 (PA5)
- new net: D13.2 (A), R44.2
- new net: Q7.2 (G), R38.1
- new net: D12.2 (A), R37.1
- new net: C15.1, D10.1 (K), U4.14 (VB3)
- new net: C14.1, D9.1 (K), U4.17 (VB2)
- new net: C13.1, D8.1 (K), U4.20 (VB1)
- new net: Q5.2 (G), R33.1
- new net: Q3.2 (G), R31.1, R32.1
- new net: Q2.2 (G), R29.1
- new net: D11.2 (A), R27.1
- new net: Q8.2 (G), R39.1, R40.1
- new net: Q6.2 (G), R34.1, R35.1
- new net: U5.1 (XTAL), Y1.1
- new net: R43.2, U5.19 (ANTB)
- new net BT_SWCLK: U5.8 (PA2)
- new net BT_SWDIO: U5.16 (PB6)
- new net U_HOUT: R29.2
- new net U_LOUT: R32.2, U4.11 (LO1)
- new net V_HOUT: R38.2, U4.16 (HO2)
- new net V_LOUT: R39.2, U4.10 (LO2)
- new net W_HOUT: R33.2, U4.13 (HO3)
- new net W_LOUT: R34.2, U4.9 (LO3)
Other:
- note added: "Bluetooth"
- note added: "Driver"
- note added: "MCU"
- note added: "可选功能"
- note added: "天线布线尽量靠近边上 周围不铺地 背面净空 元件靠近IC 晶振远离天线"
- company: (none) -> DCTek
- title: (none) -> BLDC纠编机
- moved on the sheet: C2, C8, D3, D4, D5, NTC1, NTC2, R1, R15, R16, R17, R18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

Commit message: 开环程序动起来基本可以 但是hall输出波形不对 实测HALL 需要电压高才比较稳定 但是hall信号不完整 不对称
Connections:
- net +BATT: now also R25.1
- net VDD_3.3v: no longer R25.1
Changed lines of the file:
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@@
 		)
 	)
-	(global_label "VDD_3.3v"
-		(shape input)
-		(at 276.86 135.89 90)
-		(fields_autoplaced yes)
-		(effects
-			(font
-				(size 1.27 1.27)
-			)
-			(justify left)
-		)
-		(property "Intersheetrefs" "${INTERSHEET_REFS}"
-			(at 276.86 124.3172 90)
-			(effects
-				(font
-					(size 1.27 1.27)
-				)
-				(justify left)
-				(hide yes)
-			)
-		)
-	)
 	(global_label "bemf_U"
 		(shape input)
@@
 					(unit 1)
 				)
+			)
+		)
+	)
+	(symbol
+		(lib_id "power:+BATT")
+		(at 276.86 135.89 0)
+		(unit 1)
+		(exclude_from_sim no)
+		(in_bom yes)
+		(on_board yes)
+		(dnp no)
+		(fields_autoplaced yes)
+		(property "Reference" "#PWR037"
+			(at 276.86 139.7 0)
+			(effects
+				(font
+					(size 1.27 1.27)
+				)
+				(hide yes)
+			)
+		)
+		(property "Value" "+BATT"
+			(at 276.86 130.81 0)
+			(effects
+				(font
+					(size 1.27 1.27)
+				)
+			)
+		)
+		(property "Footprint" ""
+			(at 276.86 135.89 0)
+			(effects
+				(font
+					(size 1.27 1.27)
+				)
+				(hide yes)
+			)
+		)
+		(property "Datasheet" ""
+			(at 276.86 135.89 0)
+			(effects
+				(font
+					(size 1.27 1.27)
+				)
+				(hide yes)
+			)
+		)
+		(property "Description" "Power symbol creates a global label with name \"+BATT\""
+			(at 276.86 135.89 0)
+			(effects
+				(font
+					(size 1.27 1.27)
+				)
+				(hide yes)
+			)
+		)
+		(pin "1"
+		)
+		(instances
+			(project "纠编机"
+				(path "/6ad7bea8-3496-40b6-a338-5894bb8aab93"
+					(reference "#PWR037")
+					(unit 1)
+				)
